File: hardware/kicad/esp32_m2_companion.kicad_pcb (KiCad board)
At the start: 4 copper layers, 22 x 42 mm, 33 parts, among them J1 M2_KEYB_2242_EDGE, J3 Conn_01x04, J4 Conn_01x08, U1 USBLC6-2SC6, U2 ESP32-S3-WROOM-1

Commit message: silk: add bottom-side board label + Samnium Tech logo
Name / v1.0 / Stefano Viola / 2026-08 plus the gear logomark in the top strip
(under the mounting hole, above C6/C7). Logo traced from the hi-res company
logo to smooth silk polygons (branding/gen_logo_silk.py -> logo_silk_rects.json),
applied by tools/add_silk.py (grouped 'silk_label', idempotent, never touches
copper/routing). DRC clean — only the pre-existing benign J1/GND-island notes.
Regenerated renders, 3D (GLB/STEP/STL/viewer) and datasheet views from the
silked master.

Co-Authored-By: Claude Fable 5 <noreply@anthropic.com>
Other:
- board text added: "2026-08"
- board text added: "ESP32-M2-COMPANION"
- board text added: "v1.0 Stefano Viola"
